Commit message: Fix: adjust camera_link offset to avoid self-collision in MoveIt

File: src/ur_slam_bringup/urdf/ur5e_with_camera.urdf.xacro (robot description, xacro)
@@ -170,5 +170,5 @@
     <child  link="camera_link"/>
     <!-- ツール先から少し前に出すイメージ -->
-    <origin xyz="0.0 0.0 0.01" rpy="0 0 0"/>
+    <origin xyz="0.0 0.0 0.015" rpy="0 0 0"/>
   </joint>
  <!-- Optical frames (REP-103 / REP-105 camera optical convention) -->
@@ -209,6 +209,6 @@
         </ros>
         <camera_name>depth</camera_name>
-        <image_topic_name>depth/image_raw</image_topic_name>
-        <camera_info_topic_name>depth/camera_info</camera_info_topic_name>
+        <image_topic_name>visual/image_raw</image_topic_name>
+        <camera_info_topic_name>visual/camera_info</camera_info_topic_name>
         <frame_name>camera_depth_optical_frame</frame_name>
         <publishTF>true</publishTF>

Commit message: Add ur_slam_tools package (go_to_leaf)

File: src/ur_slam_bringup/urdf/ur5e_with_camera.urdf.xacro (robot description, xacro)
@@ -154,5 +154,5 @@
       <origin xyz="0 0 0" rpy="0 0 0"/>
       <geometry>
-        <box size="0.09 0.025 0.025"/>
+        <box size="0.025 0.09 0.025"/>
       </geometry>
       <!-- 色を付けたいならここに material を追加してもOK -->
@@ -161,5 +161,5 @@
       <origin xyz="0 0 0" rpy="0 0 0"/>
       <geometry>
-        <box size="0.09 0.025 0.025"/>
+        <box size="0.025 0.09 0.025"/>
       </geometry>
     </collision>
@@ -170,5 +170,5 @@
     <child  link="camera_link"/>
     <!-- ツール先から少し前に出すイメージ -->
-    <origin xyz="0.0 0.0 0.015" rpy="0 0 0"/>
+    <origin xyz="0.0 0.0 0.015" rpy="0 -1.57079632679 1.57079632679"/>
   </joint>
  <!-- Optical frames (REP-103 / REP-105 camera optical convention) -->
@@ -200,5 +200,5 @@
         </image>
         <clip>
-          <near>0.1</near>
+          <near>0.03</near>
           <far>5.0</far>
         </clip>
@@ -226,5 +226,5 @@
         </image>
         <clip>
-          <near>0.1</near>
+          <near>0.03</near>
           <far>5.0</far>
         </clip>
